Commit message: Confirmed working MoveIt2 simulation with walls and gripper

File: src/my_ur_description/urdf/ur_system.xacro (robot description, xacro)
@@ -102,44 +102,19 @@
     <origin xyz="0 0 0" rpy="0 0 0" />
   </xacro:robotiq_gripper>
-  <ros2_control name="RobotiqGripperHardwareInterface" type="system">
+  <xacro:arg name="use_fake_hardware" default="true" />
+  <xacro:arg name="robot_ip" default="192.168.1.100" />
+  <ros2_control name="URHardwareInterface" type="system">
     <hardware>
-      <plugin>mock_components/GenericSystem</plugin>
-      <param name="calculate_dynamics">true</param>
-      <param name="mock_sensor_commands">true</param>
-    </hardware>
-    <joint name="robotiq_85_left_knuckle_joint">
-      <command_interface name="position"/>
-      <state_interface name="position"><param name="initial_value">0.0</param></state_interface>
-      <state_interface name="velocity"/>
-    </joint>
-    <joint name="robotiq_85_right_knuckle_joint">
-      <param name="mimic">robotiq_85_left_knuckle_joint</param>
-      <param name="multiplier">-1.0</param>
-      <state_interface name="position"/>
-    </joint>
-    <joint name="robotiq_85_left_inner_knuckle_joint">
-      <param name="mimic">robotiq_85_left_knuckle_joint</param>
-      <param name="multiplier">1.0</param>
-      <state_interface name="position"/>
-    </joint>
-    <joint name="robotiq_85_right_inner_knuckle_joint">
-      <param name="mimic">robotiq_85_left_knuckle_joint</param>
-      <param name="multiplier">-1.0</param>
-      <state_interface name="position"/>
-    </joint>
-    <joint name="robotiq_85_left_finger_tip_joint">
-      <param name="mimic">robotiq_85_left_knuckle_joint</param>
-      <param name="multiplier">-1.0</param> <state_interface name="position"/>
-    </joint>
-    <joint name="robotiq_85_right_finger_tip_joint">
-      <param name="mimic">robotiq_85_left_knuckle_joint</param>
-      <param name="multiplier">1.0</param>
-      <state_interface name="position"/>
-    </joint>
-  </ros2_control>
-<ros2_control name="URMockHardwareInterface" type="system">
-    <hardware>
-      <plugin>mock_components/GenericSystem</plugin>
-      <param name="calculate_dynamics">true</param>
+      <xacro:if value="$(arg use_fake_hardware)">
+        <plugin>mock_components/GenericSystem</plugin>
+        <param name="calculate_dynamics">true</param>
+      </xacro:if>
+      <xacro:unless value="$(arg use_fake_hardware)">
+        <plugin>ur_robot_driver/URPositionHardwareInterface</plugin>
+        <param name="robot_ip">$(arg robot_ip)</param>
+        <param name="script_filename">$(find ur_client_library)/resources/external_control.urscript</param>
+        <param name="output_recipe_filename">$(find ur_robot_driver)/resources/rtde_output_recipe.txt</param>
+        <param name="input_recipe_filename">$(find ur_robot_driver)/resources/rtde_input_recipe.txt</param>
+      </xacro:unless>
     </hardware>
     <joint name="shoulder_pan_joint">
@@ -174,3 +149,44 @@
     </joint>
   </ros2_control>
+  <ros2_control name="RobotiqGripperHardwareInterface" type="system">
+    <hardware>
+      <xacro:if value="$(arg use_fake_hardware)">
+        <plugin>mock_components/GenericSystem</plugin>
+      </xacro:if>
+      <xacro:unless value="$(arg use_fake_hardware)">
+        <plugin>robotiq_hardware_interface/RobotiqGripperHardwareInterface</plugin>
+        <param name="com_port">/dev/ttyUSB0</param>
+      </xacro:unless>
+    </hardware>
+    <joint name="robotiq_85_left_knuckle_joint">
+      <command_interface name="position"/>
+      <state_interface name="position"><param name="initial_value">0.0</param></state_interface>
+      <state_interface name="velocity"/>
+    </joint>
+    <joint name="robotiq_85_right_knuckle_joint">
+      <param name="mimic">robotiq_85_left_knuckle_joint</param>
+      <param name="multiplier">-1.0</param>
+      <state_interface name="position"/>
+    </joint>
+    <joint name="robotiq_85_left_inner_knuckle_joint">
+      <param name="mimic">robotiq_85_left_knuckle_joint</param>
+      <param name="multiplier">1.0</param>
+      <state_interface name="position"/>
+    </joint>
+    <joint name="robotiq_85_right_inner_knuckle_joint">
+      <param name="mimic">robotiq_85_left_knuckle_joint</param>
+      <param name="multiplier">-1.0</param>
+      <state_interface name="position"/>
+    </joint>
+    <joint name="robotiq_85_left_finger_tip_joint">
+      <param name="mimic">robotiq_85_left_knuckle_joint</param>
+      <param name="multiplier">-1.0</param>
+      <state_interface name="position"/>
+    </joint>
+    <joint name="robotiq_85_right_finger_tip_joint">
+      <param name="mimic">robotiq_85_left_knuckle_joint</param>
+      <param name="multiplier">1.0</param>
+      <state_interface name="position"/>
+    </joint>
+  </ros2_control>
 </robot>

Commit message: Modifying dimensions to be near actual physical reality

File: src/my_ur_description/urdf/ur_system.xacro (robot description, xacro)
@@ -18,5 +18,5 @@
   <joint name="world_to_desk" type="fixed">
     <parent link="world"/><child link="easydesk"/>
-    <origin xyz="0.75 0 0.9" rpy="0 0 0"/>
+    <origin xyz="0.73 0 0.9" rpy="0 0 0"/>
   </joint>
   <link name="back_wall">
@@ -88,6 +88,6 @@
     </joint>
   </xacro:macro>
-  <xacro:d435_mount prefix="cam_left" x="0.2" y="-0.4" z="0.2" yaw="1.57"/>
-  <xacro:d435_mount prefix="cam_right" x="0.6" y="-0.0" z="0.4" yaw="3.14"/>
+  <xacro:d435_mount prefix="cam_left" x="0.2" y="0.4" z="0.2" yaw="1.57"/>
+  <xacro:d435_mount prefix="cam_right" x="0.6" y="0.02" z="0.6" yaw="3.14"/>
 <xacro:ur_robot name="ur" tf_prefix="" parent="easydesk"
     joint_limits_parameters_file="$(find ur_description)/config/ur12e/joint_limits.yaml"
@@ -99,5 +99,5 @@
     safety_k_position="20"
     generate_ros2_control_tag="false">
-    <origin xyz="-0.75 0 -0.025" rpy="0 0 0" />
+    <origin xyz="-0.73 -0.05 -0.025" rpy="0 0 0" />
   </xacro:ur_robot>
   <xacro:robotiq_gripper name="robotiq_85" prefix="" parent="tool0" include_ros2_control="false">
