Commit message: correct home orientation with the real physical system

File: src/my_ur_description/srdf/ur.srdf.xacro (robot description, xacro)
@@ -19,5 +19,5 @@
   </group>
   <group_state group="ur_manipulator" name="home">
-    <joint name="$(arg prefix)shoulder_pan_joint" value="-1.5707"/>
+    <joint name="$(arg prefix)shoulder_pan_joint" value="0.0"/>
     <joint name="$(arg prefix)shoulder_lift_joint" value="-2.3562"/>
     <joint name="$(arg prefix)elbow_joint" value="2.3562"/>

File: src/my_ur_description/urdf/ur_system.xacro (robot description, xacro)
@@ -29,5 +29,5 @@
   <joint name="desk_to_back_wall" type="fixed">
     <parent link="easydesk"/><child link="back_wall"/>
-    <origin xyz="-0.25 0.6 0.75" rpy="0 0 0"/>
+    <origin xyz="-0.25 0.8 0.75" rpy="0 0 0"/>
   </joint>
   <link name="front_wall">
@@ -40,5 +40,5 @@
   <joint name="desk_to_front_wall" type="fixed">
     <parent link="easydesk"/><child link="front_wall"/>
-    <origin xyz="-0.25 -0.45 0.75" rpy="0 0 0"/>
+    <origin xyz="-0.25 -0.6 0.75" rpy="0 0 0"/>
   </joint>
   <link name="left_wall">
@@ -51,5 +51,5 @@
   <joint name="desk_to_left_wall" type="fixed">
     <parent link="easydesk"/><child link="left_wall"/>
-    <origin xyz="-1.0 0.0 0.75" rpy="0 0 0"/>
+    <origin xyz="-1.5 0.0 0.75" rpy="0 0 0"/>
   </joint>
   <link name="right_wall">
@@ -88,6 +88,6 @@
     </joint>
   </xacro:macro>
-  <xacro:d435_mount prefix="cam_left" x="0.2" y="0.4" z="0.2" yaw="1.57"/>
-  <xacro:d435_mount prefix="cam_right" x="0.6" y="0.02" z="0.6" yaw="3.14"/>
+  <xacro:d435_mount prefix="cam_left" x="0.2" y="-0.4" z="0.2" yaw="${pi/2}"/>
+  <xacro:d435_mount prefix="cam_right" x="0.6" y="0.02" z="0.6" yaw="${pi}"/>
 <xacro:ur_robot name="ur" tf_prefix="" parent="easydesk"
     joint_limits_parameters_file="$(find ur_description)/config/ur12e/joint_limits.yaml"
@@ -137,26 +137,26 @@
       <command_interface name="position"/>
       <command_interface name="velocity"/>
+      <state_interface name="position"><param name="initial_value">-2.35</param></state_interface>
+      <state_interface name="velocity"/>
+      <state_interface name="effort"/>
+    </joint>
+    <joint name="elbow_joint">
+      <command_interface name="position"/>
+      <command_interface name="velocity"/>
+      <state_interface name="position"><param name="initial_value">2.35</param></state_interface>
+      <state_interface name="velocity"/>
+      <state_interface name="effort"/>
+    </joint>
+    <joint name="wrist_1_joint">
+      <command_interface name="position"/>
+      <command_interface name="velocity"/>
       <state_interface name="position"><param name="initial_value">-1.57</param></state_interface>
       <state_interface name="velocity"/>
       <state_interface name="effort"/>
     </joint>
-    <joint name="elbow_joint">
-      <command_interface name="position"/>
-      <command_interface name="velocity"/>
-      <state_interface name="position"><param name="initial_value">0.0</param></state_interface>
-      <state_interface name="velocity"/>
-      <state_interface name="effort"/>
-    </joint>
-    <joint name="wrist_1_joint">
+    <joint name="wrist_2_joint">
       <command_interface name="position"/>
       <command_interface name="velocity"/>
       <state_interface name="position"><param name="initial_value">-1.57</param></state_interface>
-      <state_interface name="velocity"/>
-      <state_interface name="effort"/>
-    </joint>
-    <joint name="wrist_2_joint">
-      <command_interface name="position"/>
-      <command_interface name="velocity"/>
-      <state_interface name="position"><param name="initial_value">0.0</param></state_interface>
       <state_interface name="velocity"/>
       <state_interface name="effort"/>

Commit message: Again Align with real physical setup

File: src/my_ur_description/srdf/ur.srdf.xacro (robot description, xacro)
@@ -19,9 +19,9 @@
   </group>
   <group_state group="ur_manipulator" name="home">
-    <joint name="$(arg prefix)shoulder_pan_joint" value="0.0"/>
-    <joint name="$(arg prefix)shoulder_lift_joint" value="-2.3562"/>
-    <joint name="$(arg prefix)elbow_joint" value="2.3562"/>
+    <joint name="$(arg prefix)shoulder_pan_joint" value="3.1415"/>
+    <joint name="$(arg prefix)shoulder_lift_joint" value="-0.7854"/>
+    <joint name="$(arg prefix)elbow_joint" value="-2.3562"/>
     <joint name="$(arg prefix)wrist_1_joint" value="-1.5707"/>
-    <joint name="$(arg prefix)wrist_2_joint" value="-1.5707"/>
+    <joint name="$(arg prefix)wrist_2_joint" value="1.5707"/>
     <joint name="$(arg prefix)wrist_3_joint" value="0"/>
   </group_state>

File: src/my_ur_description/urdf/ur_system.xacro (robot description, xacro)
@@ -40,5 +40,5 @@
   <joint name="desk_to_front_wall" type="fixed">
     <parent link="easydesk"/><child link="front_wall"/>
-    <origin xyz="-0.25 -0.6 0.75" rpy="0 0 0"/>
+    <origin xyz="-0.25 -0.9 0.75" rpy="0 0 0"/>
   </joint>
   <link name="left_wall">
@@ -130,5 +130,5 @@
       <command_interface name="position"/>
       <command_interface name="velocity"/>
-      <state_interface name="position"><param name="initial_value">0.0</param></state_interface>
+      <state_interface name="position"><param name="initial_value">3.1415</param></state_interface>
       <state_interface name="velocity"/>
       <state_interface name="effort"/>
@@ -137,5 +137,5 @@
       <command_interface name="position"/>
       <command_interface name="velocity"/>
-      <state_interface name="position"><param name="initial_value">-2.35</param></state_interface>
+      <state_interface name="position"><param name="initial_value">-0.7854</param></state_interface>
       <state_interface name="velocity"/>
       <state_interface name="effort"/>
@@ -144,5 +144,5 @@
       <command_interface name="position"/>
       <command_interface name="velocity"/>
-      <state_interface name="position"><param name="initial_value">2.35</param></state_interface>
+      <state_interface name="position"><param name="initial_value">-2.3562</param></state_interface>
       <state_interface name="velocity"/>
       <state_interface name="effort"/>
@@ -151,5 +151,5 @@
       <command_interface name="position"/>
       <command_interface name="velocity"/>
-      <state_interface name="position"><param name="initial_value">-1.57</param></state_interface>
+      <state_interface name="position"><param name="initial_value">-1.5707</param></state_interface>
       <state_interface name="velocity"/>
       <state_interface name="effort"/>
@@ -158,5 +158,5 @@
       <command_interface name="position"/>
       <command_interface name="velocity"/>
-      <state_interface name="position"><param name="initial_value">-1.57</param></state_interface>
+      <state_interface name="position"><param name="initial_value">1.5707</param></state_interface>
       <state_interface name="velocity"/>
       <state_interface name="effort"/>

Commit message: experiment: shoulder_pan 90 deg offset adjustment for UR12e

File: src/my_ur_description/srdf/ur.srdf.xacro (robot description, xacro)
@@ -19,5 +19,5 @@
   </group>
   <group_state group="ur_manipulator" name="home">
-    <joint name="$(arg prefix)shoulder_pan_joint" value="3.1415"/>
+    <joint name="$(arg prefix)shoulder_pan_joint" value="4.7124"/>
     <joint name="$(arg prefix)shoulder_lift_joint" value="-0.7854"/>
     <joint name="$(arg prefix)elbow_joint" value="-2.3562"/>

File: src/my_ur_description/urdf/ur_system.xacro (robot description, xacro)
@@ -130,5 +130,5 @@
       <command_interface name="position"/>
       <command_interface name="velocity"/>
-      <state_interface name="position"><param name="initial_value">3.1415</param></state_interface>
+      <state_interface name="position"><param name="initial_value">4.7124</param></state_interface>
       <state_interface name="velocity"/>
       <state_interface name="effort"/>

Commit message: ur12e_new_home: apply changes for v1.1.5

File: src/my_ur_description/srdf/ur.srdf.xacro (robot description, xacro)
@@ -20,6 +20,6 @@
   <group_state group="ur_manipulator" name="home">
     <joint name="$(arg prefix)shoulder_pan_joint" value="4.7124"/>
-    <joint name="$(arg prefix)shoulder_lift_joint" value="-0.7854"/>
-    <joint name="$(arg prefix)elbow_joint" value="-2.3562"/>
+    <joint name="$(arg prefix)shoulder_lift_joint" value="-0.5236"/>
+    <joint name="$(arg prefix)elbow_joint" value="-2.618"/>
     <joint name="$(arg prefix)wrist_1_joint" value="-1.5707"/>
     <joint name="$(arg prefix)wrist_2_joint" value="1.5707"/>

File: src/my_ur_description/urdf/ur_system.xacro (robot description, xacro)
@@ -9,19 +9,30 @@
   <link name="easydesk">
     <visual>
-      <geometry><box size="1.2 0.8 0.05"/></geometry>
+      <geometry><box size="0.8 1.2 0.05"/></geometry>
       <material name="light_grey"><color rgba="0.7 0.7 0.7 1"/></material>
     </visual>
     <collision>
-      <geometry><box size="1.2 0.8 0.05"/></geometry>
+      <geometry><box size="0.8 1.2 0.05"/></geometry>
     </collision>
   </link>
   <joint name="world_to_desk" type="fixed">
     <parent link="world"/><child link="easydesk"/>
-    <origin xyz="0.73 0 0.9" rpy="0 0 0"/>
+    <origin xyz="0 0.73 0.9" rpy="0 0 0"/>
+  </joint>
+  <link name="front_wall">
+    <collision><geometry><box size="1.4 0.01 1.5"/></geometry></collision>
+    <visual>
+      <geometry><box size="1.4 0.01 1.5"/></geometry>
+      <material name="transparent_red"><color rgba="1 0 0 0.05"/></material>
+    </visual>
+  </link>
+  <joint name="desk_to_front_wall" type="fixed">
+    <parent link="easydesk"/><child link="front_wall"/>
+    <origin xyz="-0.00 0.6 0.75" rpy="0 0 0"/>
   </joint>
   <link name="back_wall">
-    <collision><geometry><box size="2.5 0.01 1.5"/></geometry></collision>
-    <visual>
-      <geometry><box size="2.5 0.01 1.5"/></geometry>
+    <collision><geometry><box size="1.4 0.01 1.5"/></geometry></collision>
+    <visual>
+      <geometry><box size="1.4 0.01 1.5"/></geometry>
       <material name="transparent_red"><color rgba="1 0 0 0.05"/></material>
     </visual>
@@ -29,21 +40,10 @@
   <joint name="desk_to_back_wall" type="fixed">
     <parent link="easydesk"/><child link="back_wall"/>
-    <origin xyz="-0.25 0.8 0.75" rpy="0 0 0"/>
-  </joint>
-  <link name="front_wall">
-    <collision><geometry><box size="2.5 0.01 1.5"/></geometry></collision>
-    <visual>
-      <geometry><box size="2.5 0.01 1.5"/></geometry>
-      <material name="transparent_red"><color rgba="1 0 0 0.05"/></material>
-    </visual>
-  </link>
-  <joint name="desk_to_front_wall" type="fixed">
-    <parent link="easydesk"/><child link="front_wall"/>
-    <origin xyz="-0.25 -0.9 0.75" rpy="0 0 0"/>
+    <origin xyz="-0.00 -1.4 0.75" rpy="0 0 0"/>
   </joint>
   <link name="left_wall">
-    <collision><geometry><box size="0.01 1.2 1.5"/></geometry></collision>
-    <visual>
-      <geometry><box size="0.01 1.2 1.5"/></geometry>
+    <collision><geometry><box size="0.01 2.25 1.5"/></geometry></collision>
+    <visual>
+      <geometry><box size="0.01 2.25 1.5"/></geometry>
       <material name="transparent_red"><color rgba="1 0 0 0.05"/></material>
     </visual>
@@ -51,10 +51,10 @@
   <joint name="desk_to_left_wall" type="fixed">
     <parent link="easydesk"/><child link="left_wall"/>
-    <origin xyz="-1.5 0.0 0.75" rpy="0 0 0"/>
+    <origin xyz="-0.6 -0.5 0.75" rpy="0 0 0"/>
   </joint>
   <link name="right_wall">
-    <collision><geometry><box size="0.01 1.2 1.5"/></geometry></collision>
-    <visual>
-      <geometry><box size="0.01 1.2 1.5"/></geometry>
+    <collision><geometry><box size="0.01 2.25 1.5"/></geometry></collision>
+    <visual>
+      <geometry><box size="0.01 2.25 1.5"/></geometry>
       <material name="transparent_red"><color rgba="1 0 0 0.05"/></material>
     </visual>
@@ -62,5 +62,5 @@
   <joint name="desk_to_right_wall" type="fixed">
     <parent link="easydesk"/><child link="right_wall"/>
-    <origin xyz="0.7 0 0.75" rpy="0 0 0"/>
+    <origin xyz="0.7 -0.5 0.75" rpy="0 0 0"/>
   </joint>
   <xacro:macro name="d435_mount" params="prefix x y z yaw">
@@ -88,6 +88,6 @@
     </joint>
   </xacro:macro>
-  <xacro:d435_mount prefix="cam_left" x="0.2" y="-0.4" z="0.2" yaw="${pi/2}"/>
-  <xacro:d435_mount prefix="cam_right" x="0.6" y="0.02" z="0.6" yaw="${pi}"/>
+  <xacro:d435_mount prefix="cam_left" x="0.4" y="+0.2" z="0.3" yaw="${pi}"/>
+  <xacro:d435_mount prefix="cam_right" x="0.02" y="0.6" z="0.6" yaw="${-pi/2}"/>
 <xacro:ur_robot name="ur" tf_prefix="" parent="easydesk"
     joint_limits_parameters_file="$(find ur_description)/config/ur12e/joint_limits.yaml"
@@ -99,5 +99,5 @@
     safety_k_position="20"
     generate_ros2_control_tag="false">
-    <origin xyz="-0.73 -0.05 -0.025" rpy="0 0 0" />
+    <origin xyz="+0.05 -0.73 -0.025" rpy="0 0 0" />
   </xacro:ur_robot>
   <xacro:robotiq_gripper name="robotiq_85" prefix="" parent="tool0" include_ros2_control="false">
@@ -137,5 +137,5 @@
       <command_interface name="position"/>
       <command_interface name="velocity"/>
-      <state_interface name="position"><param name="initial_value">-0.7854</param></state_interface>
+      <state_interface name="position"><param name="initial_value">-0.5236</param></state_interface>
       <state_interface name="velocity"/>
       <state_interface name="effort"/>
@@ -144,5 +144,5 @@
       <command_interface name="position"/>
       <command_interface name="velocity"/>
-      <state_interface name="position"><param name="initial_value">-2.3562</param></state_interface>
+      <state_interface name="position"><param name="initial_value">-2.618</param></state_interface>
       <state_interface name="velocity"/>
       <state_interface name="effort"/>
